File: ergogen/output/pcbs/boost58.kicad_pcb (KiCad board)
At the start: 2 copper layers, 147.5 x 127.5 mm, 110 parts, among them SW1 ${REFERENCE}, SW10 ${REFERENCE}, SW11 ${REFERENCE}, SW12 ${REFERENCE}, SW13 ${REFERENCE}, SW14 ${REFERENCE}, SW15 ${REFERENCE}, SW16 ${REFERENCE}, SW17 ${REFERENCE}, SW18 ${REFERENCE}, SW19 ${REFERENCE}, SW2 ${REFERENCE}, SW20 ${REFERENCE}, SW21 ${REFERENCE}, SW22 ${REFERENCE}, SW23 ${REFERENCE}, SW24 ${REFERENCE}, SW25 ${REFERENCE}, SW26 ${REFERENCE}, SW27 ${REFERENCE}, SW28 ${REFERENCE}, SW29 ${REFERENCE}, SW3 ${REFERENCE}, SW4 ${REFERENCE}, SW5 ${REFERENCE}, SW6 ${REFERENCE}, SW7 ${REFERENCE}, SW8 ${REFERENCE}, SW9 ${REFERENCE}

Commit message: re-generated PCB and drawings (will run auto-trace later)
Parts:
- D1, D10, D11, D12, D13, D14, D15, D16, D17, D18, D19, D2, D20, D21, D22, D23, D24, D25, D26, D27, D28, D29, D3, D4, D5, D6, D7, D8, D9, L1, L10, L11, L12, L13, L14, L15, L16, L17, L18, L19, L2, L20, L21, L22, L23, L24, L25, L26, L27, L28, L29, L3, L4, L5, L6, L7, L8, L9, SW1, SW10, SW11, SW12, SW13, SW14, SW15, SW16, SW17, SW18, SW19, SW2, SW20, SW21, SW22, SW23, SW24, SW25, SW26, SW27, SW28, SW29, SW3, SW4, SW5, SW6, SW7, SW8, SW9: value ${REFERENCE} -> %R
- moved UA_6 20.2 mm to (150.0, 59.0)
- moved UB_6 20.2 mm to (150.0, 66.0)
- moved M3_6 15.0 mm to (150.0, 41.0)
- moved UA_5 12.4 mm to (150.0, 97.0)
- moved UB_5 12.4 mm to (150.0, 104.0)
- moved M3_5 3.62 mm to (150.0, 115.0), turned to 0 degrees
- moved M3_1 1.00 mm to (51.0, 120.0)
- moved M3_2 1.00 mm to (51.0, 63.0)
Connections:
- SW1 pad : P1010 -> P1011
- SW10 pad : P1022 -> P1023
- SW11 pad : P1032 -> P1033
- SW12 pad : P1042 -> P1043
- SW13 pad : P1013 -> P1014
- SW14 pad : P1023 -> P1024
- SW15 pad : P1033 -> P1034
- SW16 pad : P1043 -> P1044
- SW17 pad : P1014 -> P1015
- SW18 pad : P1024 -> P1025
- SW19 pad : P1034 -> P1035
- SW2 pad : P1020 -> P1021
- SW20 pad : P1044 -> P1045
- SW21 pad : P1015 -> P1020
- SW22 pad : P1025 -> P1030
- SW23 pad : P1035 -> P1040
- SW24 pad : P1045 -> P10
- SW25 pad : P1001 -> P1002
- SW26 pad : P1002 -> P1003
- SW27 pad : P1003 -> P1004
- SW28 pad : P1004 -> P1005
- SW29 pad : P1005 -> P1010
- SW3 pad : P1030 -> P1031
- SW4 pad : P1040 -> P1041
- SW5 pad : P1011 -> P1012
- SW6 pad : P1021 -> P1022
- SW7 pad : P1031 -> P1032
- SW8 pad : P1041 -> P1042
- SW9 pad : P1012 -> P1013
Routing:
- net GND: track 1022.7 -> 96.3 mm, vias 35 -> 29
- net VCC: track 884.9 -> 96.3 mm, vias 31 -> 29
- net P6: track 241.9 -> 0.00 mm, vias 3 -> 0
- net P21: track 239.1 -> 0.00 mm
- net P5: track 230.8 -> 0.00 mm, vias 7 -> 0
- net P4: track 230.3 -> 0.00 mm, vias 7 -> 0
- net DP15: track 218.0 -> 0.00 mm, vias 2 -> 0
- net P20: track 213.0 -> 0.00 mm
- net DP19: track 206.3 -> 0.00 mm, vias 1 -> 0
- net P2: track 203.6 -> 0.00 mm, vias 5 -> 0
- net P19: track 197.7 -> 0.00 mm, vias 1 -> 0
- net DP18: track 187.7 -> 0.00 mm, vias 4 -> 0
- net P18: track 185.5 -> 0.00 mm, vias 1 -> 0
- net P3: track 183.6 -> 0.00 mm, vias 8 -> 0
- net DP14: track 181.2 -> 0.00 mm, vias 2 -> 0
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Other:
- outline, holes or cut-outs redrawn

Commit message: re-generated drawings and PCB
Parts:
- moved PWR1 20.0 mm to (172.4, 86.0)
- moved D27 0.50 mm to (119.2, 130.0)
- moved D1 0.50 mm to (40.0, 129.0)
- moved D10 0.50 mm to (80.0, 88.0)
- moved D11 0.50 mm to (80.0, 69.0)
- moved D12 0.50 mm to (80.0, 50.0)
- moved D13 0.50 mm to (100.0, 103.0)
- moved D14 0.50 mm to (100.0, 84.0)
- moved D15 0.50 mm to (100.0, 65.0)
- moved D16 0.50 mm to (100.0, 46.0)
- moved D17 0.50 mm to (120.0, 107.0)
- moved D18 0.50 mm to (120.0, 88.0)
- moved D19 0.50 mm to (120.0, 69.0)
- moved D2 0.50 mm to (40.0, 110.0)
- moved D20 0.50 mm to (120.0, 50.0)
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Other:
- board size 147.5 x 127.5 mm -> 153.6 x 133.5 mm
